Commit message: Attach two wheels to the robot

File: src/my_robot/urdf/my_robot.xacro (robot description, xacro)
@@ -51,3 +51,57 @@
         </visual>
     </link>
+    <joint name="left_wheel_joint" type="continuous">
+        <origin xyz="0.0 0.15 0.0" rpy="0.0 0.0 0.0"/>
+        <parent link="chassis"/>
+        <child link="left_wheel"/>
+        <axis xyz="0 1 0"/>
+        <limit effort="10000" velocity="1000"/>
+        <dynamic damping="1.0" friction="1.0" />
+    </joint>
+    <link name="left_wheel">
+        <inertial>
+            <origin xyz="0.0 0.0 0.0" rpy="0.0 1.5707, 1.5707"/>
+            <mass value="5.0"/>
+            <inertia ixx="0.1" ixy="0" ixz="0" iyy="0.1" iyz="0" izz="0.1" />
+        </inertial>
+        <collision>
+            <origin xyz="0.0 0.0 0.0" rpy="0.0 1.5707, 1.5707"/>
+            <geometry>
+                <cylinder radius="0.1" length="0.05"/>
+            </geometry>
+        </collision>
+        <visual name="left_wheel_visual">
+            <origin xyz="0.0 0.0 0.0" rpy="0.0 1.5707, 1.5707"/>
+            <geometry>
+                <cylinder radius="0.1" length="0.05"/>
+            </geometry>
+        </visual>
+    </link>
+    <joint name="right_wheel_joint" type="continuous">
+        <origin xyz="0.0 -0.15 0.0" rpy="0.0 0.0 0.0"/>
+        <parent link="chassis"/>
+        <child link="right_wheel"/>
+        <axis xyz="0 1 0"/>
+        <limit effort="10000" velocity="1000"/>
+        <dynamic damping="1.0" friction="1.0" />
+    </joint>
+    <link name="right_wheel">
+        <inertial>
+            <origin xyz="0.0 0.0 0.0" rpy="0.0 1.5707, 1.5707"/>
+            <mass value="5.0"/>
+            <inertia ixx="0.0" ixy="0.0" ixz="0.0" iyy="0.0" iyz="0.0" izz="0.0"/>
+        </inertial>
+        <collision>
+            <origin xyz="0.0 0.0 0.0" rpy="0.0 1.5707, 1.5707"/>
+            <geometry>
+                <cylinder radius="0.1" length="0.05"/>
+            </geometry>
+        </collision>
+        <visual name="right_wheel_visual">
+            <origin xyz="0.0 0.0 0.0" rpy="0.0 1.5707, 1.5707"/>
+            <geometry>
+                <cylinder radius="0.1" length="0.05"/>
+            </geometry>
+        </visual>
+    </link>
 </robot>

Commit message: Attach camera to robot

File: src/my_robot/urdf/my_robot.xacro (robot description, xacro)
@@ -105,3 +105,28 @@
         </visual>
     </link>
+    <joint name="camera_joint" type="fixed">
+        <origin xyz="0.2 0.0 0.0" rpy="0.0 0.0 0.0"/>
+        <parent link="chassis"/>
+        <child link="camera"/>
+        <axis xyz="0 1 0"/>
+    </joint>
+    <link name="camera">
+        <inertial>
+            <origin xyz="0.05 0.05 0.05" rpy="0.0 0.0 0.0"/>
+            <mass value="0.1"/>
+            <inertia ixx="1e-6" ixy="0" ixz="0" iyy="1e-6" iyz="0" izz="1e-6"/>
+        </inertial>
+        <collision>
+            <origin xyz="0.0 0.0 0.0" rpy="0.0 0.0 0.0"/>
+            <geometry>
+                <box size="0.05 0.05 0.05"/>
+            </geometry>
+        </collision>
+        <visual name="camera_visual">
+            <origin xyz="0.0 0.0 0.0" rpy="0.0 0.0 0.0"/>
+            <geometry>
+                <box size="0.05 0.05 0.05"/>
+            </geometry>
+        </visual>
+    </link>
 </robot>

Commit message: Add lidar

File: src/my_robot/urdf/my_robot.xacro (robot description, xacro)
@@ -125,8 +125,28 @@
         <visual name="camera_visual">
             <origin xyz="0.0 0.0 0.0" rpy="0.0 0.0 0.0"/>
+    <joint name="hokuyo_joint" type="fixed">
+        <origin xyz="0.15 0.0 0.1" rpy="0.0 0.0 0.0" />
+        <parent link="chassis" />
+        <child link="hokuyo" />
+        <axis xyz="0 1 0" />
+    </joint>
+    <link name="hokuyo">
+        <inertial>
+            <origin xyz="0.0 0.0 0.0" rpy="0.0 0.0 0.0" />
+            <mass value="1e-5" />
+            <inertia ixx="1e-6" ixy="0.0" ixz="0.0" iyy="1e-6" iyz="0.0" izz="1e-6" />
+        </inertial>
+        <visual name="hokuyo_visual">
+            <origin xyz="0.0 0.0 0.0" rpy="0.0 0.0 0.0" />
             <geometry>
-                <box size="0.05 0.05 0.05"/>
+                <mesh filename="package://my_robot/meshes/hokuyo.dae" />
             </geometry>
         </visual>
+        <collision>
+            <origin xyz="0.0 0.0 0.0" rpy="0.0 0.0 0.0" />
+            <geometry>
+                <box size="0.1 0.1 0.1" />
+            </geometry>
+        </collision>
     </link>
 </robot>

Commit message: Set robot colors

File: src/my_robot/urdf/my_robot.xacro (robot description, xacro)
@@ -2,4 +2,16 @@
 <robot name="my_robot"
     xmlns:xacro="http://www.ros.org/wiki/xacro">
+    <gazebo reference="chassis">
+        <material>Gazebo/Red</material>
+    </gazebo>
+    <gazebo reference="left_wheel">
+        <material>Gazebo/DarkYellow</material>
+    </gazebo>
+    <gazebo reference="right_wheel">
+        <material>Gazebo/DarkYellow</material>
+    </gazebo>
+    <gazebo reference="camera">
+        <material>Gazebo/DarkYellow</material>
+    </gazebo>
     <link name="robot_footprint"></link>
     <joint name="robot_footprint_joint" type="fixed">

Commit message: Format xml

File: src/my_robot/urdf/my_robot.xacro (robot description, xacro)
@@ -1,5 +1,4 @@
 <?xml version='1.0'?>
-<robot name="my_robot"
-    xmlns:xacro="http://www.ros.org/wiki/xacro">
+<robot name="my_robot" xmlns:xacro="http://www.ros.org/wiki/xacro">
     <gazebo reference="chassis">
         <material>Gazebo/Red</material>
@@ -17,124 +16,129 @@
     <joint name="robot_footprint_joint" type="fixed">
         <origin xyz="0 0 0.1" rpy="0 0 0" />
-        <parent link="robot_footprint"/>
+        <parent link="robot_footprint" />
         <child link="chassis" />
     </joint>
     <link name='chassis'>
         <inertial>
-            <mass value="15.0"/>
-            <origin xyz="0.0 0 0" rpy=" 0 0 0"/>
+            <mass value="15.0" />
+            <origin xyz="0.0 0 0" rpy=" 0 0 0" />
             <inertia ixx="0.1" ixy="0" ixz="0" iyy="0.1" iyz="0" izz="0.1" />
         </inertial>
         <collision name='collision'>
-            <origin xyz="0 0 0" rpy=" 0 0 0"/>
+            <origin xyz="0 0 0" rpy=" 0 0 0" />
             <geometry>
-                <box size=".4 .2 .1"/>
+                <box size=".4 .2 .1" />
             </geometry>
         </collision>
         <visual name='chassis_visual'>
-            <origin xyz="0 0 0" rpy=" 0 0 0"/>
+            <origin xyz="0 0 0" rpy=" 0 0 0" />
             <geometry>
-                <box size=".4 .2 .1"/>
+                <box size=".4 .2 .1" />
             </geometry>
         </visual>
         <collision name='back_caster_collision'>
-            <origin xyz="-0.15 0 -0.05" rpy=" 0 0 0"/>
+            <origin xyz="-0.15 0 -0.05" rpy=" 0 0 0" />
             <geometry>
-                <sphere radius="0.0499"/>
+                <sphere radius="0.0499" />
             </geometry>
         </collision>
         <visual name='back_caster_visual'>
-            <origin xyz="-0.15 0 -0.05" rpy=" 0 0 0"/>
+            <origin xyz="-0.15 0 -0.05" rpy=" 0 0 0" />
             <geometry>
-                <sphere radius="0.05"/>
+                <sphere radius="0.05" />
             </geometry>
         </visual>
         <collision name='front_caster_collision'>
-            <origin xyz="0.15 0 -0.05" rpy=" 0 0 0"/>
+            <origin xyz="0.15 0 -0.05" rpy=" 0 0 0" />
             <geometry>
-                <sphere radius="0.0499"/>
+                <sphere radius="0.0499" />
             </geometry>
         </collision>
         <visual name='front_caster_visual'>
-            <origin xyz="0.15 0 -0.05" rpy=" 0 0 0"/>
+            <origin xyz="0.15 0 -0.05" rpy=" 0 0 0" />
             <geometry>
-                <sphere radius="0.05"/>
+                <sphere radius="0.05" />
             </geometry>
         </visual>
     </link>
     <joint name="left_wheel_joint" type="continuous">
-        <origin xyz="0.0 0.15 0.0" rpy="0.0 0.0 0.0"/>
-        <parent link="chassis"/>
-        <child link="left_wheel"/>
-        <axis xyz="0 1 0"/>
-        <limit effort="10000" velocity="1000"/>
+        <origin xyz="0.0 0.15 0.0" rpy="0.0 0.0 0.0" />
+        <parent link="chassis" />
+        <child link="left_wheel" />
+        <axis xyz="0 1 0" />
+        <limit effort="10000" velocity="1000" />
         <dynamic damping="1.0" friction="1.0" />
     </joint>
     <link name="left_wheel">
         <inertial>
-            <origin xyz="0.0 0.0 0.0" rpy="0.0 1.5707, 1.5707"/>
-            <mass value="5.0"/>
+            <origin xyz="0.0 0.0 0.0" rpy="0.0 1.5707, 1.5707" />
+            <mass value="5.0" />
             <inertia ixx="0.1" ixy="0" ixz="0" iyy="0.1" iyz="0" izz="0.1" />
         </inertial>
         <collision>
-            <origin xyz="0.0 0.0 0.0" rpy="0.0 1.5707, 1.5707"/>
+            <origin xyz="0.0 0.0 0.0" rpy="0.0 1.5707, 1.5707" />
             <geometry>
-                <cylinder radius="0.1" length="0.05"/>
+                <cylinder radius="0.1" length="0.05" />
             </geometry>
         </collision>
         <visual name="left_wheel_visual">
-            <origin xyz="0.0 0.0 0.0" rpy="0.0 1.5707, 1.5707"/>
+            <origin xyz="0.0 0.0 0.0" rpy="0.0 1.5707, 1.5707" />
             <geometry>
-                <cylinder radius="0.1" length="0.05"/>
+                <cylinder radius="0.1" length="0.05" />
             </geometry>
         </visual>
     </link>
     <joint name="right_wheel_joint" type="continuous">
-        <origin xyz="0.0 -0.15 0.0" rpy="0.0 0.0 0.0"/>
-        <parent link="chassis"/>
-        <child link="right_wheel"/>
-        <axis xyz="0 1 0"/>
-        <limit effort="10000" velocity="1000"/>
+        <origin xyz="0.0 -0.15 0.0" rpy="0.0 0.0 0.0" />
+        <parent link="chassis" />
+        <child link="right_wheel" />
+        <axis xyz="0 1 0" />
+        <limit effort="10000" velocity="1000" />
         <dynamic damping="1.0" friction="1.0" />
     </joint>
     <link name="right_wheel">
         <inertial>
-            <origin xyz="0.0 0.0 0.0" rpy="0.0 1.5707, 1.5707"/>
-            <mass value="5.0"/>
-            <inertia ixx="0.0" ixy="0.0" ixz="0.0" iyy="0.0" iyz="0.0" izz="0.0"/>
+            <origin xyz="0.0 0.0 0.0" rpy="0.0 1.5707, 1.5707" />
+            <mass value="5.0" />
+            <inertia ixx="0.0" ixy="0.0" ixz="0.0" iyy="0.0" iyz="0.0" izz="0.0" />
         </inertial>
         <collision>
-            <origin xyz="0.0 0.0 0.0" rpy="0.0 1.5707, 1.5707"/>
+            <origin xyz="0.0 0.0 0.0" rpy="0.0 1.5707, 1.5707" />
             <geometry>
-                <cylinder radius="0.1" length="0.05"/>
+                <cylinder radius="0.1" length="0.05" />
             </geometry>
         </collision>
         <visual name="right_wheel_visual">
-            <origin xyz="0.0 0.0 0.0" rpy="0.0 1.5707, 1.5707"/>
+            <origin xyz="0.0 0.0 0.0" rpy="0.0 1.5707, 1.5707" />
             <geometry>
-                <cylinder radius="0.1" length="0.05"/>
+                <cylinder radius="0.1" length="0.05" />
             </geometry>
         </visual>
     </link>
     <joint name="camera_joint" type="fixed">
-        <origin xyz="0.2 0.0 0.0" rpy="0.0 0.0 0.0"/>
-        <parent link="chassis"/>
-        <child link="camera"/>
-        <axis xyz="0 1 0"/>
+        <origin xyz="0.2 0.0 0.0" rpy="0.0 0.0 0.0" />
+        <parent link="chassis" />
+        <child link="camera" />
+        <axis xyz="0 1 0" />
     </joint>
     <link name="camera">
         <inertial>
-            <origin xyz="0.05 0.05 0.05" rpy="0.0 0.0 0.0"/>
-            <mass value="0.1"/>
-            <inertia ixx="1e-6" ixy="0" ixz="0" iyy="1e-6" iyz="0" izz="1e-6"/>
+            <origin xyz="0.05 0.05 0.05" rpy="0.0 0.0 0.0" />
+            <mass value="0.1" />
+            <inertia ixx="1e-6" ixy="0" ixz="0" iyy="1e-6" iyz="0" izz="1e-6" />
         </inertial>
         <collision>
-            <origin xyz="0.0 0.0 0.0" rpy="0.0 0.0 0.0"/>
+            <origin xyz="0.0 0.0 0.0" rpy="0.0 0.0 0.0" />
             <geometry>
-                <box size="0.05 0.05 0.05"/>
+                <box size="0.05 0.05 0.05" />
             </geometry>
         </collision>
         <visual name="camera_visual">
-            <origin xyz="0.0 0.0 0.0" rpy="0.0 0.0 0.0"/>
+            <origin xyz="0.0 0.0 0.0" rpy="0.0 0.0 0.0" />
+            <geometry>
+                <box size="0.05 0.05 0.05" />
+            </geometry>
+        </visual>
+    </link>
     <joint name="hokuyo_joint" type="fixed">
         <origin xyz="0.15 0.0 0.1" rpy="0.0 0.0 0.0" />

Commit message: Fix right wheel inertia

File: src/my_robot/urdf/my_robot.xacro (robot description, xacro)
@@ -101,5 +101,5 @@
             <origin xyz="0.0 0.0 0.0" rpy="0.0 1.5707, 1.5707" />
             <mass value="5.0" />
-            <inertia ixx="0.0" ixy="0.0" ixz="0.0" iyy="0.0" iyz="0.0" izz="0.0" />
+            <inertia ixx="0.1" ixy="0" ixz="0" iyy="0.1" iyz="0" izz="0.1" />
         </inertial>
         <collision>

Commit message: Increase chassis width from .2 to .3

File: src/my_robot/urdf/my_robot.xacro (robot description, xacro)
@@ -28,5 +28,5 @@
             <origin xyz="0 0 0" rpy=" 0 0 0" />
             <geometry>
-                <box size=".4 .2 .1" />
+                <box size=".4 .3 .1" />
             </geometry>
         </collision>
@@ -34,5 +34,5 @@
             <origin xyz="0 0 0" rpy=" 0 0 0" />
             <geometry>
-                <box size=".4 .2 .1" />
+                <box size=".4 .3 .1" />
             </geometry>
         </visual>
@@ -63,5 +63,5 @@
     </link>
     <joint name="left_wheel_joint" type="continuous">
-        <origin xyz="0.0 0.15 0.0" rpy="0.0 0.0 0.0" />
+        <origin xyz="0.0 0.2 0.0" rpy="0.0 0.0 0.0" />
         <parent link="chassis" />
         <child link="left_wheel" />
@@ -90,5 +90,5 @@
     </link>
     <joint name="right_wheel_joint" type="continuous">
-        <origin xyz="0.0 -0.15 0.0" rpy="0.0 0.0 0.0" />
+        <origin xyz="0.0 -0.2 0.0" rpy="0.0 0.0 0.0" />
         <parent link="chassis" />
         <child link="right_wheel" />

Commit message: Increase wheel size

File: src/my_robot/urdf/my_robot.xacro (robot description, xacro)
@@ -15,5 +15,5 @@
     <link name="robot_footprint"></link>
     <joint name="robot_footprint_joint" type="fixed">
-        <origin xyz="0 0 0.1" rpy="0 0 0" />
+        <origin xyz="0 0 0.125" rpy="0 0 0" />
         <parent link="robot_footprint" />
         <child link="chassis" />
@@ -28,5 +28,5 @@
             <origin xyz="0 0 0" rpy=" 0 0 0" />
             <geometry>
-                <box size=".4 .3 .1" />
+                <box size=".55 .3 .1" />
             </geometry>
         </collision>
@@ -34,5 +34,5 @@
             <origin xyz="0 0 0" rpy=" 0 0 0" />
             <geometry>
-                <box size=".4 .3 .1" />
+                <box size=".55 .3 .1" />
             </geometry>
         </visual>
@@ -40,5 +40,5 @@
             <origin xyz="-0.15 0 -0.05" rpy=" 0 0 0" />
             <geometry>
-                <sphere radius="0.0499" />
+                <sphere radius="0.075" />
             </geometry>
         </collision>
@@ -46,5 +46,5 @@
             <origin xyz="-0.15 0 -0.05" rpy=" 0 0 0" />
             <geometry>
-                <sphere radius="0.05" />
+                <sphere radius="0.075" />
             </geometry>
         </visual>
@@ -52,5 +52,5 @@
             <origin xyz="0.15 0 -0.05" rpy=" 0 0 0" />
             <geometry>
-                <sphere radius="0.0499" />
+                <sphere radius="0.075" />
             </geometry>
         </collision>
@@ -58,5 +58,5 @@
             <origin xyz="0.15 0 -0.05" rpy=" 0 0 0" />
             <geometry>
-                <sphere radius="0.05" />
+                <sphere radius="0.075" />
             </geometry>
         </visual>
@@ -79,5 +79,5 @@
             <origin xyz="0.0 0.0 0.0" rpy="0.0 1.5707, 1.5707" />
             <geometry>
-                <cylinder radius="0.1" length="0.05" />
+                <cylinder radius="0.125" length="0.05" />
             </geometry>
         </collision>
@@ -85,5 +85,5 @@
             <origin xyz="0.0 0.0 0.0" rpy="0.0 1.5707, 1.5707" />
             <geometry>
-                <cylinder radius="0.1" length="0.05" />
+                <cylinder radius="0.125" length="0.05" />
             </geometry>
         </visual>
@@ -106,5 +106,5 @@
             <origin xyz="0.0 0.0 0.0" rpy="0.0 1.5707, 1.5707" />
             <geometry>
-                <cylinder radius="0.1" length="0.05" />
+                <cylinder radius="0.125" length="0.05" />
             </geometry>
         </collision>
@@ -112,10 +112,10 @@
             <origin xyz="0.0 0.0 0.0" rpy="0.0 1.5707, 1.5707" />
             <geometry>
-                <cylinder radius="0.1" length="0.05" />
+                <cylinder radius="0.125" length="0.05" />
             </geometry>
         </visual>
     </link>
     <joint name="camera_joint" type="fixed">
-        <origin xyz="0.2 0.0 0.0" rpy="0.0 0.0 0.0" />
+        <origin xyz="0.3 0.0 0.0" rpy="0.0 0.0 0.0" />
         <parent link="chassis" />
         <child link="camera" />
@@ -142,5 +142,5 @@
     </link>
     <joint name="hokuyo_joint" type="fixed">
-        <origin xyz="0.15 0.0 0.1" rpy="0.0 0.0 0.0" />
+        <origin xyz="0.25 0.0 0.1" rpy="0.0 0.0 0.0" />
         <parent link="chassis" />
         <child link="hokuyo" />

Commit message: Add horns

File: src/my_robot/urdf/my_robot.xacro (robot description, xacro)
@@ -12,4 +12,10 @@
     <gazebo reference="camera">
         <material>Gazebo/DarkYellow</material>
+    </gazebo>
+    <gazebo reference="left_front_horn">
+        <material>Gazebo/Gold</material>
+    </gazebo>
+    <gazebo reference="right_front_horn">
+        <material>Gazebo/Gold</material>
     </gazebo>
     <link name="robot_footprint"></link>
@@ -166,3 +172,53 @@
         </collision>
     </link>
+    <joint name="left_front_horn_joint" type="fixed">
+        <origin xyz="0.27 0.13 0.0" rpy="0.0 0.0 0.0" />
+        <parent link="chassis" />
+        <child link="left_front_horn" />
+        <axis xyz="0 1 0" />
+    </joint>
+    <link name="left_front_horn">
+        <inertial>
+            <origin xyz="0.15 0.0 0.0" rpy="0.0 0.0 0.0" />
+            <mass value="0.1" />
+            <inertia ixx="1e-6" ixy="0" ixz="0" iyy="1e-6" iyz="0" izz="1e-6" />
+        </inertial>
+        <collision name="left_front_horn_collision">
+            <origin xyz="0.15 0.0 0.0" rpy="0.0 0.0 0.0" />
+            <geometry>
+                <box size="0.3 0.02 0.05" />
+            </geometry>
+        </collision>
+        <visual name="left_front_horn_visual">
+            <origin xyz="0.15 0.0 0.0" rpy="0.0 0.0 0.0" />
+            <geometry>
+                <box size="0.3 0.02 0.05" />
+            </geometry>
+        </visual>
+    </link>
+    <joint name="right_front_horn_joint" type="fixed">
+        <origin xyz="0.27 -0.13 0.0" rpy="0.0 0.0 0.0" />
+        <parent link="chassis" />
+        <child link="right_front_horn" />
+        <axis xyz="0 1 0" />
+    </joint>
+    <link name="right_front_horn">
+        <inertial>
+            <origin xyz="0.15 0.0 0.0" rpy="0.0 0.0 0.0" />
+            <mass value="0.1" />
+            <inertia ixx="1e-6" ixy="0" ixz="0" iyy="1e-6" iyz="0" izz="1e-6" />
+        </inertial>
+        <collision name="right_front_horn_collision">
+            <origin xyz="0.15 0.0 0.0" rpy="0.0 0.0 0.0" />
+            <geometry>
+                <box size="0.3 0.02 0.05" />
+            </geometry>
+        </collision>
+        <visual name="right_front_horn_visual">
+            <origin xyz="0.15 0.0 0.0" rpy="0.0 0.0 0.0" />
+            <geometry>
+                <box size="0.3 0.02 0.05" />
+            </geometry>
+        </visual>
+    </link>
 </robot>

Commit message: Rename wheel joints

File: src/my_robot/urdf/my_robot.xacro (robot description, xacro)
@@ -68,5 +68,5 @@
         </visual>
     </link>
-    <joint name="left_wheel_joint" type="continuous">
+    <joint name="left_wheel_hinge" type="continuous">
         <origin xyz="0.0 0.2 0.0" rpy="0.0 0.0 0.0" />
         <parent link="chassis" />
@@ -95,5 +95,5 @@
         </visual>
     </link>
-    <joint name="right_wheel_joint" type="continuous">
+    <joint name="right_wheel_hinge" type="continuous">
         <origin xyz="0.0 -0.2 0.0" rpy="0.0 0.0 0.0" />
         <parent link="chassis" />

Commit message: Fix wheel inertial

File: src/my_robot/urdf/my_robot.xacro (robot description, xacro)
@@ -70,8 +70,8 @@
     </link>
     <joint name="left_wheel_hinge" type="continuous">
-        <origin xyz="0.0 0.2 0.0" rpy="0.0 0.0 0.0" />
+        <origin xyz="0 0.2 0" rpy="0 0 0" />
         <parent link="chassis" />
         <child link="left_wheel" />
-        <axis xyz="0 1 0" />
+        <axis xyz="0 1 0" rpy="0 0 0" />
         <limit effort="10000" velocity="1000" />
         <dynamic damping="1.0" friction="1.0" />
@@ -79,10 +79,10 @@
     <link name="left_wheel">
         <inertial>
-            <origin xyz="0.0 0.0 0.0" rpy="0.0 1.5707, 1.5707" />
+            <origin xyz="0 0 0" rpy="0 1.5707 1.5707" />
             <mass value="5.0" />
             <inertia ixx="0.1" ixy="0" ixz="0" iyy="0.1" iyz="0" izz="0.1" />
         </inertial>
         <collision>
-            <origin xyz="0.0 0.0 0.0" rpy="0.0 1.5707, 1.5707" />
+            <origin xyz="0 0 0" rpy="0 1.5707 1.5707" />
             <geometry>
                 <cylinder radius="0.125" length="0.05" />
@@ -90,5 +90,5 @@
         </collision>
         <visual name="left_wheel_visual">
-            <origin xyz="0.0 0.0 0.0" rpy="0.0 1.5707, 1.5707" />
+            <origin xyz="0 0 0" rpy="0 1.5707 1.5707" />
             <geometry>
                 <cylinder radius="0.125" length="0.05" />
@@ -106,10 +106,10 @@
     <link name="right_wheel">
         <inertial>
-            <origin xyz="0.0 0.0 0.0" rpy="0.0 1.5707, 1.5707" />
+            <origin xyz="0.0 0.0 0.0" rpy="0.0 1.5707 1.5707" />
             <mass value="5.0" />
             <inertia ixx="0.1" ixy="0" ixz="0" iyy="0.1" iyz="0" izz="0.1" />
         </inertial>
         <collision>
-            <origin xyz="0.0 0.0 0.0" rpy="0.0 1.5707, 1.5707" />
+            <origin xyz="0.0 0.0 0.0" rpy="0.0 1.5707 1.5707" />
             <geometry>
                 <cylinder radius="0.125" length="0.05" />
@@ -117,5 +117,5 @@
         </collision>
         <visual name="right_wheel_visual">
-            <origin xyz="0.0 0.0 0.0" rpy="0.0 1.5707, 1.5707" />
+            <origin xyz="0.0 0.0 0.0" rpy="0.0 1.5707 1.5707" />
             <geometry>
                 <cylinder radius="0.125" length="0.05" />
