Commit message: Fix world file

File: src/my_robot/urdf/my_robot.xacro (robot description, xacro)
@@ -29,9 +29,9 @@
         <inertial>
             <mass value="15.0" />
-            <origin xyz="0.0 0 0" rpy=" 0 0 0" />
+            <origin xyz="0 0 0" rpy="0 0 0" />
             <inertia ixx="0.1" ixy="0" ixz="0" iyy="0.1" iyz="0" izz="0.1" />
         </inertial>
         <collision name='collision'>
-            <origin xyz="0 0 0" rpy=" 0 0 0" />
+            <origin xyz="0 0 0" rpy="0 0 0" />
             <geometry>
                 <box size=".55 .3 .1" />
@@ -39,5 +39,5 @@
         </collision>
         <visual name='chassis_visual'>
-            <origin xyz="0 0 0" rpy=" 0 0 0" />
+            <origin xyz="0 0 0" rpy="0 0 0" />
             <geometry>
                 <box size=".55 .3 .1" />

Commit message: Change robot initial position

File: src/my_robot/urdf/my_robot.xacro (robot description, xacro)
@@ -22,5 +22,5 @@
     <link name="robot_footprint"></link>
     <joint name="robot_footprint_joint" type="fixed">
-        <origin xyz="0 0 0.125" rpy="0 0 0" />
+        <origin xyz="-2 -3 0.125" rpy="0 0 0" />
         <parent link="robot_footprint" />
         <child link="chassis" />

Commit message: Revert "Change robot initial position"
This reverts commit 6ce697fc08d75f3ec76cbab2ca5233e2cc31c19c.

File: src/my_robot/urdf/my_robot.xacro (robot description, xacro)
@@ -22,5 +22,5 @@
     <link name="robot_footprint"></link>
     <joint name="robot_footprint_joint" type="fixed">
-        <origin xyz="-2 -3 0.125" rpy="0 0 0" />
+        <origin xyz="0 0 0.125" rpy="0 0 0" />
         <parent link="robot_footprint" />
         <child link="chassis" />

Commit message: Adjust horn size

File: src/my_robot/urdf/my_robot.xacro (robot description, xacro)
@@ -181,18 +181,18 @@
     <link name="left_front_horn">
         <inertial>
-            <origin xyz="0.15 0.0 0.0" rpy="0.0 0.0 0.0" />
+            <origin xyz="0.0 0.0 0.0" rpy="0.0 0.0 0.0" />
             <mass value="0.1" />
             <inertia ixx="1e-6" ixy="0" ixz="0" iyy="1e-6" iyz="0" izz="1e-6" />
         </inertial>
         <collision name="left_front_horn_collision">
-            <origin xyz="0.15 0.0 0.0" rpy="0.0 0.0 0.0" />
-            <geometry>
-                <box size="0.3 0.02 0.05" />
+            <origin xyz="0.0 0.0 0.0" rpy="0.0 0.0 0.0" />
+            <geometry>
+                <box size="0.2 0.02 0.05" />
             </geometry>
         </collision>
         <visual name="left_front_horn_visual">
-            <origin xyz="0.15 0.0 0.0" rpy="0.0 0.0 0.0" />
-            <geometry>
-                <box size="0.3 0.02 0.05" />
+            <origin xyz="0.0 0.0 0.0" rpy="0.0 0.0 0.0" />
+            <geometry>
+                <box size="0.2 0.02 0.05" />
             </geometry>
         </visual>
@@ -206,18 +206,18 @@
     <link name="right_front_horn">
         <inertial>
-            <origin xyz="0.15 0.0 0.0" rpy="0.0 0.0 0.0" />
+            <origin xyz="0.0 0.0 0.0" rpy="0.0 0.0 0.0" />
             <mass value="0.1" />
             <inertia ixx="1e-6" ixy="0" ixz="0" iyy="1e-6" iyz="0" izz="1e-6" />
         </inertial>
         <collision name="right_front_horn_collision">
-            <origin xyz="0.15 0.0 0.0" rpy="0.0 0.0 0.0" />
-            <geometry>
-                <box size="0.3 0.02 0.05" />
+            <origin xyz="0.0 0.0 0.0" rpy="0.0 0.0 0.0" />
+            <geometry>
+                <box size="0.2 0.02 0.05" />
             </geometry>
         </collision>
         <visual name="right_front_horn_visual">
-            <origin xyz="0.15 0.0 0.0" rpy="0.0 0.0 0.0" />
-            <geometry>
-                <box size="0.3 0.02 0.05" />
+            <origin xyz="0.0 0.0 0.0" rpy="0.0 0.0 0.0" />
+            <geometry>
+                <box size="0.2 0.02 0.05" />
             </geometry>
         </visual>
